File: pcb/USB_JTAG.sch (KiCad schematic (older format))
At the start: 26 parts, among them J1 JVWW9, P1 DF3_6, U1 Q6CVQ, U2 JPPQ9, U3 26HRB, U4 6DXQ7, U5 B4CF9

Commit message: fix FT232 FP
Parts:
- removed C8: 1 uF, kicad_pcb:0402, symbol capacitors:capacitor_0402
- removed D1: QF838, 0603_led, symbol diode:QF838
- removed J1: JVWW9, kicad_pcb:USB_micro_B, symbol connector:JVWW9
- removed P1: DF3_6, kicad_pcb:DF3_6, symbol connector:TC2030-NL
- removed U4: 6DXQ7, kicad_pcb:SC70-5, symbol ic:6DXQ7
- removed U5: B4CF9, kicad_pcb:QFN32_5x5_4V, symbol ic:B4CF9
- added J1: USBC_China16, kicad_pcb:USB_C_Receptacle_China_16pin, symbol connector:USBC_China16
- added J2: Conn_01x08_Male, Connector_Hirose:Hirose_DF13-08P-1.25DSA_1x08_P1.25mm_Vertical, symbol Connector:Conn_01x08_Male
- added R7: 5.1 k, kicad_pcb:R_0402_1005Metric, symbol resistor:resistor_0402
- added R8, R9: 499, kicad_pcb:R_0402_1005Metric, symbol resistor:resistor_0402
- added U4, U5, U6, U8: 6MMF7, kicad_pcb:SOT-363_SC-70-6, symbol ic:6MMF7
- C1, C10, C2, C3, C5, C6, C7, C9: footprint kicad_pcb:0402 -> kicad_pcb:C_0402_1005Metric
- C4: footprint kicad_pcb:0805 -> kicad_pcb:C_0805_2012Metric
- R1, R2, R3, R4, R5: footprint kicad_pcb:0402_R -> kicad_pcb:R_0402_1005Metric
- R6: value 1 k -> 5.1 k; footprint kicad_pcb:0402_R -> kicad_pcb:R_0402_1005Metric; Power (none) -> 0.05
- TH1, TH2: footprint tooling_hole_2.55 -> kicad_pcb:tooling_hole_2.55
- U1: footprint kicad_pcb:SOT23-6 -> kicad_pcb:SOT-23-6
- U2: footprint osc_2.5x2 -> kicad_pcb:Oscillator_SMD_4Pin_2.5x2.0mm
- U3: footprint kicad_pcb:QFN48_7x7 -> kicad_pcb:QFN-48-1EP_8x8mm_P0.5mm_EP6.2x6.2mm
Connections:
- net labels added: CC1, CC2, DIR, TCK2, TDI1, TDO1, TDO2, TMS1
- net labels removed: 1V2, ACBUS3, ACBUS4, ACBUS7, ACBUS8, ADBUS4, CRESET, F_CLK, F_CS, F_DI, F_DO, LED0, LED1
- wire segments 106 -> 123
- no-connect marks 17 -> 16
Other:
- moved on the sheet: C10, R5

Commit message: fix TDI/TDO swap closes #2
Connections:
- net TDI: now also J2.7 (Pin_7), R8.2, U8.4 (B); no longer J2.4 (Pin_4), J2.5 (Pin_5), U4.4 (B)
- net TDI1: now also R9.2; no longer U4.3 (A)
- net TDO: now also J2.4 (Pin_4), J2.5 (Pin_5), U4.4 (B); no longer J2.7 (Pin_7), R8.2, U8.4 (B)
- net TDO1: now also U4.3 (A); no longer R9.2
- net TDO2 renamed TDI2
Changed lines of the file:
@@
 Sheet 1 1
 Title "USB to JTAG and SWD interface"
-Date "2018-10-16"
-Rev "4"
+Date "2019-06-19"
+Rev "5.1"
 Comp "Harmon Instruments, LLC"
 Comment1 "Licensed under GNU GPL 3.0 or later"
@@
 	5250 6500 5250 6600
 Wire Wire Line
-	6300 3200 5600 3200
+	6300 3300 5600 3300
 Wire Wire Line
 	3550 6100 3550 6000
@@
 Text Label 5700 3100 0    50   ~ 0
 TCK1
+Text Label 5700 3300 0    50   ~ 0
+TDO1
 Text Label 5700 3200 0    50   ~ 0
 TDI1
-Text Label 5700 3300 0    50   ~ 0
-TDO1
 Text Label 5700 3400 0    50   ~ 0
 TMS1
@@
 TCK2
 Text Label 8450 4950 0    50   ~ 0
-TDO
+TDI
 $Comp
 L combined:+3.3V #PWR09
@@
 $EndComp
 Wire Wire Line
-	6200 3300 5600 3300
+	6200 3200 5600 3200
 Wire Wire Line
 	7400 3100 7950 3100
@@
 	7800 6000 9100 6000
 Text Label 8250 4100 0    50   ~ 0
-TDI
+TDO
 Wire Wire Line
 	7950 4500 7500 4500
@@
 	7000 4950 6750 4950
 Wire Wire Line
-	6200 3300 6200 4950
+	6200 3200 6200 4950
 Wire Wire Line
 	7500 3700 7500 4500
@@
 Wire Wire Line
 	6300 4100 6550 4100
-Wire Wire Line
-	6300 3200 6300 4100
 $Comp
 L resistor:resistor_0402 R9
@@
 	6250 4950 6200 4950
 Text Label 6800 4950 0    50   ~ 0
-TDO2
+TDI2
 Wire Wire Line
 	7000 5150 6000 5150
@@
 Text Label 6650 5150 0    50   ~ 0
 DIR
+Wire Wire Line
+	6300 3300 6300 4100
 $EndSCHEMATC

Commit message: Fix net labels closes #3
Parts:
- J1: value USBC_China16 -> CGH8B; footprint kicad_pcb:USB_C_Receptacle_China_16pin -> kicad_pcb:USB_C_Receptacle_HRO_TYPE-C-31-M-12; symbol connector:USBC_China16 -> connector:CGH8B
Connections:
- net TDI: now also J2.4 (Pin_4), J2.5 (Pin_5), U4.4 (B); no longer J2.7 (Pin_7), R8.2, U8.4 (B)
- net TDI1: now also U3.15 (ADBUS2_DI), U4.3 (A); no longer R9.2, U3.14 (ADBUS1_DO)
- net TDO: now also J2.7 (Pin_7), R8.2, U8.4 (B); no longer J2.4 (Pin_4), J2.5 (Pin_5), U4.4 (B)
- net TDO1: now also R9.2, U3.14 (ADBUS1_DO); no longer U3.15 (ADBUS2_DI), U4.3 (A)
- net TDI2 renamed TDO2
Changed lines of the file:
@@
 EESchema Schematic File Version 4
 LIBS:USB_JTAG-cache
-EELAYER 29 0
+EELAYER 30 0
 EELAYER END
 $Descr USLetter 11000 8500
@@
 TCK1
 Text Label 5700 3300 0    50   ~ 0
+TDI1
+Text Label 5700 3200 0    50   ~ 0
 TDO1
-Text Label 5700 3200 0    50   ~ 0
-TDI1
 Text Label 5700 3400 0    50   ~ 0
 TMS1
@@
 TCK2
 Text Label 8450 4950 0    50   ~ 0
-TDI
+TDO
 $Comp
 L combined:+3.3V #PWR09
@@
 	7950 5600 7500 5600
 $Comp
-L connector:USBC_China16 J1
-U 1 1 5CFBB2A7
-P 1000 3250
-F 0 "J1" H 883 3415 50  0000 C CNN
-F 1 "USBC_China16" H 883 3324 50  0000 C CNN
-F 2 "kicad_pcb:USB_C_Receptacle_China_16pin" H 600 3300 50  0001 L CNN
-F 3 "$PARTS/8RYXT/SJ117928.pdf" V 850 3250 50  0001 C CNN
-	1    1000 3250
-	1    0    0    -1
-$EndComp
-$Comp
 L combined:ground #GND0101
 U 1 1 5CFBDC24
@@
 	7800 6000 9100 6000
 Text Label 8250 4100 0    50   ~ 0
-TDO
+TDI
 Wire Wire Line
 	7950 4500 7500 4500
@@
 	6250 4950 6200 4950
 Text Label 6800 4950 0    50   ~ 0
-TDI2
+TDO2
 Wire Wire Line
 	7000 5150 6000 5150
@@
 Wire Wire Line
 	6300 3300 6300 4100
+$Comp
+L connector:CGH8B J1
+U 1 1 5CFBB2A7
+P 1000 3250
+F 0 "J1" H 883 3415 50  0000 C CNN
+F 1 "CGH8B" H 883 3324 50  0000 C CNN
+F 2 "kicad_pcb:USB_C_Receptacle_HRO_TYPE-C-31-M-12" H 600 3300 50  0001 L CNN
+F 3 "${PARTS}/CGH8B/TYPE-C-31-M-12.pdf" V 850 3250 50  0001 C CNN
+	1    1000 3250
+	1    0    0    -1
+$EndComp
 $EndSCHEMATC
